File: kabeer_neurotech_afe/neurotech_afe/neurotech_afe.kicad_sch (KiCad schematic)
At the start: 27 parts, among them J1 Conn_01x03_Pin, U1 AD620, U2 Opamp_Quad

Commit message: digipots
Parts:
- removed R11: 12.35k, symbol Device:R
- removed R2: 26.5k, symbol Device:R
- removed R3: 5.86k, symbol Device:R
- removed R4, R8: 10k, symbol Device:R
- removed R5, R6: 10.6k, symbol Device:R
- removed R7: 5.86, symbol Device:R
- removed U1: AD620, symbol Amplifier_Instrumentation:AD620
- added 10k? (x2): R_Small, symbol Device:R_Small
- added 50k, 5k: R_Potentiometer_Dual, symbol Device:R_Potentiometer_Dual
- added R?: 510, symbol Device:R
- added U?: AD8226ARZ, R_8_ADI, symbol Components:AD8226ARZ
- C2: value 10nF -> 22nF
- C4: value 1uF -> 2.2uF
- R1: value 26.5k -> 10k
Connections:
- net +3.3V: now also U?.8 (VS+)
- net 1.65 V: now also C2.2, 5k.2, U?.6 (REF)
- net GND: now also U?.5 (VS-); no longer C2.2
- net at C1.1: now also 50k.3, 50k.5; no longer R1.2
- net at C1.2, C3.1, U2.1: now also U2.2 (-)
- net at C2.1, U2.3 (+): now also 50k.6
- net at C3.2, C4.1: now also 10k?.1
- net at C4.2, U2.5 (+): now also 10k?.1
- net In+: now reaches D1.3 (COM), R15.2, R18.1
- net In+: now also U?.4 (IN+)
- net at U2.6 (-): now also U2.10 (+), U2.7, 10k?.2, 5k.5
- net In-: now reaches D2.3 (COM), R14.2, R16.1
- net In-: now also U?.1 (IN-)
- net IAout: now reaches R1.1
- net IAout: now also U?.7 (VOUT)
- new net: 50k.2, R1.2
- new net: 10k?.2, 5k.3
- new net: R?.1, U?.3 (RG)
- new net: R?.2, U?.2 (RG)
- no-connect marks 0 -> 4
Other:
- moved on the sheet: C1, C2, J1, R1, R10, R12, R13, R17, R9, U2A, U2D, U2E
