File: finalKiCad/neurotech_afe.kicad_sch (KiCad schematic)
At the start: 33 parts, among them J1 Conn_01x02_Pin, U1 ADS1220xPW, U2 Opamp_Quad, U3 MCP4141T-103E/SN, U4 TLV70033_SOT23-5, U5 AD8226ARZ, U6 EXB24V332JX, U7 113991054, U8 EXB34V105JV

Commit message: routing
Parts:
- R4: footprint Resistor_SMD:R_0201_0603Metric_Pad0.64x0.40mm_HandSolder -> Resistor_SMD:R_0603_1608Metric_Pad0.98x0.95mm_HandSolder
Changed lines of the file:
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@@
 			)
 		)
-		(property "Footprint" "Resistor_SMD:R_0201_0603Metric_Pad0.64x0.40mm_HandSolder"
+		(property "Footprint" "Resistor_SMD:R_0603_1608Metric_Pad0.98x0.95mm_HandSolder"
 			(at 347.98 58.42 0)
 			(effects
