File: finalKiCad/neurotech_afe.kicad_pcb (KiCad board)
At the start: 2 copper layers, 27 parts, among them U1 ADS1220xPW, U2 Opamp_Quad, U4 TLV70033_SOT23-5, U5 AD8226ARZ

Commit message: footprints and started layout
Parts:
- removed 10k1: R_Small, Resistor_SMD:R_0201_0603Metric_Pad0.64x0.40mm_HandSolder
- removed D1, D2: BAT54S, Package_TO_SOT_SMD:SOT-23
- added J1: Conn_01x02_Pin, Flex-EMG:BATT_CONN, F.Cu at (137.5, 129.3)
- added R3: 10k, Resistor_SMD:R_0603_1608Metric_Pad0.98x0.95mm_HandSolder, F.Cu at (206.3, 67.4)
- added R4: 3.3k, Resistor_SMD:R_0201_0603Metric_Pad0.64x0.40mm_HandSolder, F.Cu at (208.5, 82.2)
- added R5: 20k, Flex-EMG:POT_PTN16-A20120K1B1, F.Cu at (224.9, 70.6)
- added R6: 50k, Flex-EMG:POT_PTN16-A20120K1B1, F.Cu at (225.0, 89.1)
- added U3: MCP4141T-103E/SN, Flex-EMG:SOIC8-N_MC_MCH, F.Cu at (210.4, 77.6)
- added U6: EXB24V332JX, Flex-EMG:C_ARRAY_EXB24V_PAN, F.Cu at (167.2, 85.2)
- added U7: 113991054, Flex-EMG:ESP32C3, F.Cu at (175.9, 128.7)
- added U8: EXB34V105JV, Flex-EMG:C_ARRAY_EXB34V_PAN, F.Cu at (171.1, 85.1)
- C1, C10, C11, C12, C2, C3, C4, C5, C6, C8, C9: footprint Capacitor_SMD:C_0201_0603Metric_Pad0.64x0.40mm_HandSolder -> Capacitor_SMD:C_0603_1608Metric_Pad1.08x0.95mm_HandSolder
- C7: value C -> 4.7n; footprint Capacitor_SMD:C_0201_0603Metric_Pad0.64x0.40mm_HandSolder -> Capacitor_SMD:C_0603_1608Metric_Pad1.08x0.95mm_HandSolder
- R1, R12, R13, R17: footprint Resistor_SMD:R_0201_0603Metric_Pad0.64x0.40mm_HandSolder -> Resistor_SMD:R_0603_1608Metric_Pad0.98x0.95mm_HandSolder
- R2: footprint Resistor_SMD:R_0201_0603Metric_Pad0.64x0.40mm_HandSolder -> Resistor_SMD:R_0603_1608Metric_Pad0.98x0.95mm_HandSolder; moved to B.Cu
- TP1, TP2, TP3: footprint TestPoint:TestPoint_THTPad_D2.0mm_Drill1.0mm -> TestPoint:TestPoint_THTPad_D4.0mm_Drill2.0mm
- U1: footprint Package_SO:TSSOP-16_4.4x5mm_P0.65mm -> Flex-EMG:SOP65P640X120-16N
- U2: footprint Package_SO:SOIC-14_3.9x8.7mm_P1.27mm -> Flex-EMG:SOP65P640X120-14N
- moved C3 113.4 mm to (206.3, 65.5), turned to 180 degrees
- moved C10 106.9 mm to (201.4, 121.7), turned to 180 degrees
- moved C2 106.4 mm to (202.3, 88.1)
- moved C1 98.2 mm to (201.0, 71.2)
- moved C4 97.9 mm to (208.9, 66.5), turned to 90 degrees
- moved R17 97.4 mm to (193.4, 59.3)
- moved R1 88.2 mm to (201.2, 68.8), turned to 180 degrees
- moved C11 86.7 mm to (201.4, 114.4), turned to 180 degrees
- moved C12 78.1 mm to (186.8, 58.7)
- moved U2 72.9 mm to (209.6, 71.6)
- moved C9 72.0 mm to (149.3, 127.8), turned to -90 degrees
- moved U4 70.6 mm to (146.3, 128.8)
- moved C8 70.1 mm to (143.0, 129.4), turned to 90 degrees
- moved C5 62.6 mm to (175.3, 79.0), turned to -90 degrees
- moved C6 61.5 mm to (173.6, 79.0), turned to -90 degrees
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Connections:
- C2 pad 2: /Vout -> /1.65 V
- U2 pad 9: /Vout -> Net-(U2C--)
Routing:
- net GND: track 6.47 -> 39.3 mm, vias 3 -> 5
- net +3.3V: track 1.48 -> 20.0 mm, vias 0 -> 1
- net /In-: track 0.00 -> 13.3 mm
- net /1.65 V: track 1.27 -> 8.63 mm, vias 0 -> 1
- net Net-(U2B--): track 6.75 -> 0.00 mm
- net /In+: track 0.00 -> 6.22 mm
- net Net-(U2D-+): track 3.91 -> 0.00 mm
- net Net-(R2-Pad2): track 0.00 -> 3.61 mm, vias 0 -> 1
- net Net-(R2-Pad1): track 0.00 -> 3.45 mm, vias 0 -> 1
- net /3V7: track 10.4 -> 12.1 mm, vias 0 -> 3
- net Net-(U2A--): track 1.27 -> 2.73 mm
- net /Vout: track 1.27 -> 0.00 mm
- removed copper zone on B.Cu, net GND
Other:
- copper layers 2 -> 4

Commit message: routing
Parts:
- R4: footprint Resistor_SMD:R_0201_0603Metric_Pad0.64x0.40mm_HandSolder -> Resistor_SMD:R_0603_1608Metric_Pad0.98x0.95mm_HandSolder
- moved R17 60.1 mm to (187.1, 119.0), turned to 180 degrees
- moved R13 56.2 mm to (183.4, 116.7), turned to 180 degrees
- moved C7 56.0 mm to (196.1, 126.2), turned to 90 degrees
- moved C12 55.9 mm to (187.7, 114.5), turned to -90 degrees
- moved R2 53.1 mm to (193.6, 126.0), turned to -90 degrees
- moved C5 52.4 mm to (189.2, 129.5), turned to 0 degrees
- moved U5 50.4 mm to (190.8, 126.0), turned to 180 degrees
- moved C4 50.0 mm to (197.6, 115.2), turned to -90 degrees
- moved C6 49.6 mm to (186.2, 127.1), turned to 90 degrees
- moved U2 47.0 mm to (192.6, 115.4), turned to 180 degrees
- moved C3 46.9 mm to (199.9, 111.9), turned to -90 degrees
- moved U6 44.2 mm to (192.5, 121.5), turned to 180 degrees
- moved R3 44.1 mm to (197.7, 110.6), turned to 90 degrees
- moved R12 43.7 mm to (183.4, 114.9), turned to 180 degrees
- moved R1 41.6 mm to (193.6, 109.7)
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Routing:
- net /SCLK: track 0.00 -> 54.4 mm, vias 0 -> 1
- net /DIN: track 0.00 -> 53.0 mm, vias 0 -> 1
- net /Vout: track 0.00 -> 38.3 mm
- net /DOUT: track 0.00 -> 22.4 mm
- net /CS: track 0.00 -> 11.2 mm, vias 0 -> 2
- net Net-(U2B--): track 0.00 -> 10.9 mm
- net GND: track 39.3 -> 29.9 mm, vias 5 -> 6
- net Net-(U2D-+): track 0.00 -> 9.09 mm
- net Net-(U2B-+): track 0.00 -> 7.21 mm
- net Net-(R4-Pad2): track 0.00 -> 5.67 mm
- net Net-(U2C--): track 0.00 -> 5.06 mm
- net Net-(C3-Pad2): track 0.00 -> 5.02 mm
- net /1.65 V: track 8.63 -> 12.7 mm
- net /DRDY: track 0.00 -> 3.98 mm
- net +3.3V: track 20.0 -> 23.0 mm, vias 1 -> 4
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
Commit message: silkscreen
Parts:
- removed TP1, TP2, TP3: TestPoint, TestPoint:TestPoint_THTPad_D4.0mm_Drill2.0mm
- added G***: LOGO, LOGO, F.Cu at (162.6, 135.0)
- added J2: B3B-PH-K-S, Flex-EMG:JST_B3B-PH-K-S, F.Cu at (178.5, 133.5)
- added TP4: TestPoint, TestPoint:TestPoint_THTPad_D4.0mm_Drill2.0mm, F.Cu at (182.2, 139.5)
- added TP5: TestPoint, TestPoint:TestPoint_THTPad_D4.0mm_Drill2.0mm, F.Cu at (175.6, 139.6)
- R4: moved to B.Cu
- moved R5 66.4 mm to (165.1, 116.2), turned to -90 degrees
- moved R6 66.4 mm to (164.9, 97.9), turned to -90 degrees
- moved J1 63.0 mm to (164.7, 72.9), turned to 0 degrees
- moved C10 55.9 mm to (162.4, 82.1), turned to 180 degrees
- moved C6 55.9 mm to (161.4, 77.0), turned to 0 degrees
- moved C8 54.9 mm to (164.8, 76.9), turned to 0 degrees
- moved U7 50.2 mm to (178.9, 78.6), turned to 0 degrees
- moved U4 49.7 mm to (164.6, 79.5), turned to 180 degrees
- moved C9 49.6 mm to (161.5, 79.6), turned to 90 degrees
- moved U1 40.6 mm to (180.6, 95.1), turned to -90 degrees
- moved C12 39.1 mm to (165.9, 82.1), turned to 0 degrees
- moved C1 21.7 mm to (173.3, 103.7), turned to 90 degrees
- moved C3 21.5 mm to (178.5, 112.7), turned to 90 degrees
- moved C4 21.4 mm to (176.4, 112.7), turned to 90 degrees
- moved R1 20.5 mm to (173.3, 107.3), turned to 90 degrees
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Connections:
- U8 pad 1: /In- -> /In+
- U8 pad 2: /In+ -> /In-
Routing:
- net /CS1: track 0.00 -> 35.3 mm, vias 0 -> 1
- net /Vout: track 38.3 -> 6.36 mm
- net /1.65 V: track 12.7 -> 42.8 mm, vias 1 -> 6
- net /DRDY: track 3.98 -> 33.4 mm, vias 0 -> 1
- net /SCLK: track 54.4 -> 24.9 mm, vias 1 -> 2
- net /DIN: track 53.0 -> 27.4 mm, vias 1 -> 5
- net /CS: track 11.2 -> 30.3 mm, vias 2 -> 1
- net Net-(U2A-+): track 2.14 -> 20.6 mm
- net GND: track 29.9 -> 43.8 mm, vias 6 -> 43
- net Net-(U2B-+): track 7.21 -> 20.3 mm
- net Net-(C1-Pad1): track 1.85 -> 10.8 mm
- net +3.3V: track 23.0 -> 30.6 mm, vias 4 -> 16
- net Net-(U2A--): track 2.78 -> 8.58 mm
- net Net-(U2D-+): track 9.09 -> 3.81 mm
- net /Reference_Electrode: track 0.00 -> 5.07 mm
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- added copper zone on In2.Cu, net +3.3V
- added copper zone on In2.Cu, net /1.65 V
- added copper zone on In2.Cu, net /3V7
- added copper zone on In1.Cu, net GND
Other:
- board outline added: 35.3 x 75.7 mm
- board text added: "GND"
- board text added: "NT@B Flex-EMG Sp' 26 Alex Wong Sean Isomatsu Leo Ragogna Abhay Dharnidharka Kabeer Nayyar Edgar Amezcua"
- board text added: "Power"
